Commit message: finished portion of 4dof urdf

File: install/four_dof/share/four_dof/urdf/draft.urdf (robot description, URDF)
Before this commit: robot four_dof, 3 links, 2 joints
Links:
- added link left_foot; collision mesh filename=package://four_dof/meshes/left_foot.stl scale=0.001 0.001 0.001; visual mesh filename=package://four_dof/meshes/left_foot.stl scale=0.001 0.001 0.001
- added link left_front_knee; collision mesh filename=package://four_dof/meshes/left_front_knee_link.stl scale=0.001 0.001 0.001; visual mesh filename=package://four_dof/meshes/left_front_knee_link.stl scale=0.001 0.001 0.001
- added link right_foot; collision mesh filename=package://four_dof/meshes/right_foot.stl scale=0.001 0.001 0.001; visual mesh filename=package://four_dof/meshes/right_foot.stl scale=0.001 0.001 0.001
- added link right_front_knee; collision mesh filename=package://four_dof/meshes/right_front_knee_link.stl scale=0.001 0.001 0.001; visual mesh filename=package://four_dof/meshes/right_front_knee_link.stl scale=0.001 0.001 0.001
- added link right_front_thigh; collision mesh filename=package://four_dof/meshes/right_front_thigh_link.stl scale=0.001 0.001 0.001; visual mesh filename=package://four_dof/meshes/right_front_thigh_link.stl scale=0.001 0.001 0.001
Joints:
- added joint body_to_right_thigh: type revolute, parent body, child right_front_thigh, origin xyz=0.035 0.0165 -0.05125 rpy=0 0 0, axis 0.0 0.0 1, limit lower=-1.57 upper=1.57 effort=1000.0 velocity=0.5
- added joint left_knee_to_foot: type revolute, parent left_front_knee, child left_foot, origin xyz=0.0 -0.110041 0.0 rpy=0.0 0.0 -1.57, axis 0.0 0.0 1.0, limit lower=1.57 upper=1.57 effort=0.0 velocity=0.0
- added joint left_thigh_to_knee: type revolute, parent left_front_thigh, child left_front_knee, origin xyz=0.0 -0.1335 0.01835 rpy=0 0 0, axis 0.0 0.0 1, limit lower=-1.57 upper=1.57 effort=0 velocity=0
- added joint right_knee_to_foot: type revolute, parent right_front_knee, child right_foot, origin xyz=0.0 -0.110041 0.0 rpy=0.0 0.0 -1.57, axis 0.0 0.0 1.0, limit lower=1.57 upper=1.57 effort=0.0 velocity=0.0
- added joint right_thigh_to_knee: type revolute, parent right_front_thigh, child right_front_knee, origin xyz=0.0 -0.1335 0.01835 rpy=0 0 0, axis 0.0 0.0 1, limit lower=-1.57 upper=1.57 effort=0 velocity=0
- joint base_to_body: origin xyz=0 0 0 rpy=1.57 0 0  -> xyz=0.0 0.0 0 rpy=1.57 0 0 

Commit message: drafted a new urdf, with inertial

File: install/four_dof/share/four_dof/urdf/draft.urdf (robot description, URDF)
Before this commit: robot four_dof, 8 links, 7 joints
Links:
- link body: mass None -> 1.1161; geometry collision mesh filename=package://four_dof/meshes/draft1/body_for_Sym.stl scale=0.001 0.001 0.001; visual mesh filename=package://four_dof/meshes/draft1/body_for_Sym.stl scale=0.001 0.001 0.001
- link left_foot: geometry collision mesh filename=package://four_dof/meshes/draft1/left_foot.stl scale=0.001 0.001 0.001; visual mesh filename=package://four_dof/meshes/draft1/left_foot.stl scale=0.001 0.001 0.001
- link left_front_knee: geometry collision mesh filename=package://four_dof/meshes/draft1/left_front_knee_link.stl scale=0.001 0.001 0.001; visual mesh filename=package://four_dof/meshes/draft1/left_front_knee_link.stl scale=0.001 0.001 0.001
- link left_front_thigh: geometry collision mesh filename=package://four_dof/meshes/draft1/left_front_thigh_link.stl scale=0.001 0.001 0.001; visual mesh filename=package://four_dof/meshes/draft1/left_front_thigh_link.stl scale=0.001 0.001 0.001
- link right_foot: geometry collision mesh filename=package://four_dof/meshes/draft1/right_foot.stl scale=0.001 0.001 0.001; visual mesh filename=package://four_dof/meshes/draft1/right_foot.stl scale=0.001 0.001 0.001
- link right_front_knee: geometry collision mesh filename=package://four_dof/meshes/draft1/right_front_knee_link.stl scale=0.001 0.001 0.001; visual mesh filename=package://four_dof/meshes/draft1/right_front_knee_link.stl scale=0.001 0.001 0.001
- link right_front_thigh: geometry collision mesh filename=package://four_dof/meshes/draft1/right_front_thigh_link.stl scale=0.001 0.001 0.001; visual mesh filename=package://four_dof/meshes/draft1/right_front_thigh_link.stl scale=0.001 0.001 0.001
