Commit message: six dof bot added

File: install/four_dof/share/four_dof/urdf/draft2.urdf (robot description, URDF)
Before this commit: robot four_dof, 8 links, 7 joints
Joints:
- joint body_to_left_thigh: limit lower=-1.57 upper=1.57 effort=1000.0 velocity=0.5 -> lower=-0.26 upper=0.52 effort=35.0 velocity=0.1
- joint body_to_right_thigh: limit lower=-1.57 upper=1.57 effort=1000.0 velocity=0.5 -> lower=-0.26 upper=0.52 effort=35.0 velocity=0.1
- joint left_knee_to_foot: limit lower=-1.57 upper=1.57 effort=1000 velocity=0 -> lower=-0.3 upper=0.3 effort=35 velocity=0; origin xyz=0.0 -0.110041 0.0 rpy=0.0 0.0 -1.57 -> xyz=0.0 -0.110041 0.0 rpy=0.0 0.0 0
- joint left_thigh_to_knee: limit lower=-1.57 upper=1.57 effort=1000 velocity=0 -> lower=-0.52 upper=0.52 effort=35 velocity=0.1
- joint right_knee_to_foot: limit lower=-1.57 upper=1.57 effort=1000 velocity=0 -> lower=-0.3 upper=0.3 effort=35 velocity=0; origin xyz=0.0 -0.110041 0.0 rpy=0.0 0.0 -1.57 -> xyz=0.0 -0.110041 0.0 rpy=0.0 0.0 0
- joint right_thigh_to_knee: limit lower=-1.57 upper=1.57 effort=1000 velocity=0 -> lower=-0.52 upper=0.52 effort=35 velocity=0.1
