Commit message: added lateral joints

File: install/six_dof/share/six_dof/urdf/6dof_fixed.urdf (robot description, URDF)
Before this commit: robot 6dof, 7 links, 6 joints
Links:
- added link intermediate_link
- link body: geometry collision mesh filename=package://six_dof/meshes/chassisv2.stl scale=0.001 0.001 0.001; visual mesh filename=package://six_dof/meshes/chassisv2.stl scale=0.001 0.001 0.001
- link left_foot: geometry collision mesh filename=package://six_dof/meshes/leftfootfixed.stl scale=0.001 0.001 0.001; visual mesh filename=package://six_dof/meshes/leftfootfixed.stl scale=0.001 0.001 0.001
- link left_shin: geometry collision mesh filename=package://six_dof/meshes/rightshinv3.stl scale=0.001 0.001 0.001; visual mesh filename=package://six_dof/meshes/rightshinv3.stl scale=0.001 0.001 0.001
- link right_foot: geometry collision mesh filename=package://six_dof/meshes/leftfootfixed.stl scale=0.001 0.001 0.001; visual mesh filename=package://six_dof/meshes/leftfootfixed.stl scale=0.001 0.001 0.001
- link right_shin: geometry collision mesh filename=package://six_dof/meshes/rightshinv4.stl scale=0.01 0.01 0.01; visual mesh filename=package://six_dof/meshes/rightshinv4.stl scale=0.01 0.01 0.01
- link right_thigh: geometry collision mesh filename=package://six_dof/meshes/rightthighfixedv1.stl scale=0.001 0.001 0.001; visual mesh filename=package://six_dof/meshes/rightthighfixedv1.stl scale=0.001 0.001 0.001
Joints:
- added joint body_left_thigh_lateral: type revolute, parent body, child left_thigh, origin xyz=0.100 0 0 rpy=0 3.14 0, axis  0 0 1, limit lower=-0.15 upper=0.15 effort=35.0 velocity=0.1
- added joint right_thigh_body_lateral: type revolute, parent intermediate_link, child body, origin xyz=0 0 0 rpy=0 0 0, axis  0 0 1, limit lower=-0.15 upper=0.15 effort=35.0 velocity=0.1
- joint body_left_thigh: limit lower=-0.26 upper=0.52 effort=35.0 velocity=0.1 -> lower=-0.52 upper=0.69 effort=35.0 velocity=0.1; origin xyz=0.100 0 0 rpy=0 3.14 0 -> xyz=0 0 0 rpy=0 0 0
- joint left_shin_foot: limit lower=-0.26 upper=0.52 effort=35.0 velocity=0.1 -> lower=-0.52 upper=0.52 effort=35.0 velocity=0.1; origin xyz=-0.022 -0.130 0 rpy=-1.57 0 0 -> xyz=-0.022 -0.130 0 rpy=-1.57 3.14 0
- joint left_thigh_shin: limit lower=-0.26 upper=0.52 effort=35.0 velocity=0.1 -> lower=-0.52 upper=0.52 effort=35.0 velocity=0.1
- joint right_foot_shin: limit lower=-0.26 upper=0.52 effort=35.0 velocity=0.1 -> lower=-0.52 upper=0.52 effort=35.0 velocity=0.1; origin xyz=0.005 0.025 0.0265 rpy=1.57 0 0 -> xyz=0.004 0.0 0.0 rpy=1.57 0 0
- joint right_shin_thigh: limit lower=-0.26 upper=0.52 effort=35.0 velocity=0.1 -> lower=-0.52 upper=0.52 effort=35.0 velocity=0.1
- joint right_thigh_body: child body -> intermediate_link; limit lower=-0.26 upper=0.52 effort=35.0 velocity=0.1 -> lower=-0.69 upper=0.52 effort=35.0 velocity=0.1

File: src/six_dof/urdf/6dof_fixed.urdf (robot description, URDF)
Before this commit: robot 6dof, 7 links, 6 joints
Links:
- added link intermediate_link
- link body: geometry collision mesh filename=package://six_dof/meshes/chassisv2.stl scale=0.001 0.001 0.001; visual mesh filename=package://six_dof/meshes/chassisv2.stl scale=0.001 0.001 0.001
- link left_foot: geometry collision mesh filename=package://six_dof/meshes/leftfootfixed.stl scale=0.001 0.001 0.001; visual mesh filename=package://six_dof/meshes/leftfootfixed.stl scale=0.001 0.001 0.001
- link left_shin: geometry collision mesh filename=package://six_dof/meshes/rightshinv3.stl scale=0.001 0.001 0.001; visual mesh filename=package://six_dof/meshes/rightshinv3.stl scale=0.001 0.001 0.001
- link right_foot: geometry collision mesh filename=package://six_dof/meshes/leftfootfixed.stl scale=0.001 0.001 0.001; visual mesh filename=package://six_dof/meshes/leftfootfixed.stl scale=0.001 0.001 0.001
- link right_shin: geometry collision mesh filename=package://six_dof/meshes/rightshinv4.stl scale=0.01 0.01 0.01; visual mesh filename=package://six_dof/meshes/rightshinv4.stl scale=0.01 0.01 0.01
- link right_thigh: geometry collision mesh filename=package://six_dof/meshes/rightthighfixedv1.stl scale=0.001 0.001 0.001; visual mesh filename=package://six_dof/meshes/rightthighfixedv1.stl scale=0.001 0.001 0.001
Joints:
- added joint body_left_thigh_lateral: type revolute, parent body, child left_thigh, origin xyz=0.100 0 0 rpy=0 3.14 0, axis  0 0 1, limit lower=-0.15 upper=0.15 effort=35.0 velocity=0.1
- added joint right_thigh_body_lateral: type revolute, parent intermediate_link, child body, origin xyz=0 0 0 rpy=0 0 0, axis  0 0 1, limit lower=-0.15 upper=0.15 effort=35.0 velocity=0.1
- joint body_left_thigh: limit lower=-0.26 upper=0.52 effort=35.0 velocity=0.1 -> lower=-0.52 upper=0.69 effort=35.0 velocity=0.1; origin xyz=0.100 0 0 rpy=0 3.14 0 -> xyz=0 0 0 rpy=0 0 0
- joint left_shin_foot: limit lower=-0.26 upper=0.52 effort=35.0 velocity=0.1 -> lower=-0.52 upper=0.52 effort=35.0 velocity=0.1; origin xyz=-0.022 -0.130 0 rpy=-1.57 0 0 -> xyz=-0.022 -0.130 0 rpy=-1.57 3.14 0
- joint left_thigh_shin: limit lower=-0.26 upper=0.52 effort=35.0 velocity=0.1 -> lower=-0.52 upper=0.52 effort=35.0 velocity=0.1
- joint right_foot_shin: limit lower=-0.26 upper=0.52 effort=35.0 velocity=0.1 -> lower=-0.52 upper=0.52 effort=35.0 velocity=0.1; origin xyz=0.005 0.025 0.0265 rpy=1.57 0 0 -> xyz=0.004 0.0 0.0 rpy=1.57 0 0
- joint right_shin_thigh: limit lower=-0.26 upper=0.52 effort=35.0 velocity=0.1 -> lower=-0.52 upper=0.52 effort=35.0 velocity=0.1
- joint right_thigh_body: child body -> intermediate_link; limit lower=-0.26 upper=0.52 effort=35.0 velocity=0.1 -> lower=-0.69 upper=0.52 effort=35.0 velocity=0.1

Commit message: updated gitignore, fixed intermediate link issue in body to left thigh

File: install/six_dof/share/six_dof/urdf/6dof_fixed.urdf (robot description, URDF)
Before this commit: robot 6dof, 8 links, 8 joints
Links:
- added link intermediate_link_2
Joints:
- joint body_left_thigh: parent body -> intermediate_link_2
- joint body_left_thigh_lateral: child left_thigh -> intermediate_link_2

Commit message: fixed joint limits

File: install/six_dof/share/six_dof/urdf/6dof_fixed.urdf (robot description, URDF)
Before this commit: robot 6dof, 9 links, 8 joints
Joints:
- joint body_left_thigh: limit lower=-0.52 upper=0.69 effort=35.0 velocity=0.1 -> lower=-0.78 upper=1.57 effort=35.0 velocity=0.1
- joint body_left_thigh_lateral: limit lower=-0.15 upper=0.15 effort=35.0 velocity=0.1 -> lower=-0.26 upper=0.26 effort=35.0 velocity=0.1
- joint right_thigh_body: limit lower=-0.69 upper=0.52 effort=35.0 velocity=0.1 -> lower=-0.78 upper=1.57 effort=35.0 velocity=0.1
- joint right_thigh_body_lateral: limit lower=-0.15 upper=0.15 effort=35.0 velocity=0.1 -> lower=-0.26 upper=0.26 effort=35.0 velocity=0.1

File: src/six_dof/urdf/6dof_test.urdf (robot description, URDF)
Before this commit: robot 6dof, 9 links, 8 joints
Joints:
- joint body_left_thigh: limit lower=-0.78 upper=1.57 effort=35.0 velocity=0.1 -> lower=-0.52 upper=0.69 effort=35.0 velocity=0.1
- joint body_left_thigh_lateral: limit lower=-0.26 upper=0.26 effort=35.0 velocity=0.1 -> lower=-0.15 upper=0.15 effort=35.0 velocity=0.1
- joint left_shin_foot: axis  1 0 0 -> (none); limit lower=-0.52 upper=0.52 effort=35.0 velocity=0.1 -> (none); type revolute -> fixed
- joint right_foot_shin: axis  1 0 0 -> (none); limit lower=-0.52 upper=0.52 effort=35.0 velocity=0.1 -> (none); type revolute -> fixed
- joint right_thigh_body: limit lower=-0.78 upper=1.57 effort=35.0 velocity=0.1 -> lower=-0.69 upper=0.52 effort=35.0 velocity=0.1
- joint right_thigh_body_lateral: limit lower=-0.26 upper=0.26 effort=35.0 velocity=0.1 -> lower=-0.15 upper=0.15 effort=35.0 velocity=0.1
