Commit message: added a fixed foot urdf, and modified base link of existing urdf

File: src/six_dof/urdf/6dof_from_hip_fixed.urdf (robot description, URDF)
Before this commit: robot 6dof, 10 links, 9 joints
Joints:
- joint base_body: origin xyz=0.0 0.050 0.3095 rpy=1.57 0.0 0.0 -> xyz=0.0 0.0 0.0 rpy=1.57 0.0 0.0
- joint left_shin_foot: axis  1 0 0 -> (none); limit lower=-0.52 upper=0.52 effort=35.0 velocity=0.1 -> (none); type revolute -> fixed
- joint right_shin_foot: axis  1 0 0 -> (none); limit lower=-0.52 upper=0.52 effort=35.0 velocity=0.1 -> (none); type revolute -> fixed
