Commit message: added new urdf from hip and associated mesh files

File: src/six_dof/urdf/6dof_from_hip.urdf (robot description, URDF)
Before this commit: robot 6dof, 10 links, 9 joints
Links:
- link right_shin: geometry collision mesh filename=package://six_dof/meshes/rightshinfixedv2.stl scale=0.001 0.001 0.001; visual mesh filename=package://six_dof/meshes/rightshinfixedv2.stl scale=0.001 0.001 0.001
- link right_thigh: geometry collision mesh filename=package://six_dof/meshes/rightthighfixedv2.stl scale=0.001 0.001 0.001; visual mesh filename=package://six_dof/meshes/rightthighfixedv2.stl scale=0.001 0.001 0.001
Joints:
- joint left_shin_foot: origin xyz=-0.022 -0.130 0 rpy=-1.57 3.14 0 -> xyz=-0.027 -0.130 0 rpy=-1.57 3.14 0
- joint right_body_thigh: limit lower=-0.78 upper=1.57 effort=35.0 velocity=0.1 -> lower=-1.57 upper=0.78 effort=35.0 velocity=0.1; origin xyz=0.041 -0.160 0 rpy=0 0 0 -> xyz=0.041 0 0 rpy=0 0 0
- joint right_shin_foot: origin xyz=-0.004 0.0 0.0 rpy=-1.57 0 0 -> xyz=-0.02 -0.130 0.0 rpy=-1.57 0 0
- joint right_thigh_shin: origin xyz=-0.0125 -0.130 0 rpy=0 0 0 -> xyz=0.0025 -0.160 0 rpy=0 0 0

Commit message: added flat feet

File: src/six_dof/urdf/6dof_from_hip.urdf (robot description, URDF)
Before this commit: robot 6dof, 10 links, 9 joints
Links:
- link left_foot: geometry collision mesh filename=package://six_dof/meshes/foot_fixedv2.stl scale=0.001 0.001 0.001; visual mesh filename=package://six_dof/meshes/foot_fixedv2.stl scale=0.001 0.001 0.001
- link right_foot: geometry collision mesh filename=package://six_dof/meshes/foot_fixedv2.stl scale=0.001 0.001 0.001; visual mesh filename=package://six_dof/meshes/foot_fixedv2.stl scale=0.001 0.001 0.001
Joints:
- joint left_shin_foot: origin xyz=-0.027 -0.130 0 rpy=-1.57 3.14 0 -> xyz=-0.027 -0.130 0 rpy=-1.57 1.57 0
- joint right_shin_foot: origin xyz=-0.02 -0.130 0.0 rpy=-1.57 0 0 -> xyz=-0.02 -0.130 0.0 rpy=-1.57 -1.57 0

Commit message: modififed CMake to find pinocchio eigen and include eigen

File: src/six_dof/urdf/6dof_from_hip.urdf (robot description, URDF)
Before this commit: robot 6dof, 10 links, 9 joints
Joints:
- joint left_shin_foot: origin xyz=-0.027 -0.130 0 rpy=-1.57 1.57 0 -> xyz=-0.027 -0.130 0 rpy=0 0 0
- joint right_shin_foot: origin xyz=-0.02 -0.130 0.0 rpy=-1.57 -1.57 0 -> xyz=-0.02 -0.130 0.0 rpy=0 0 0

Commit message: final urdf

File: src/six_dof/urdf/6dof_from_hip.urdf (robot description, URDF)
Before this commit: robot 6dof, 10 links, 9 joints
Links:
- link left_foot: geometry collision mesh filename=package://six_dof/meshes/footfixedv3.stl scale=0.001 0.001 0.001; visual mesh filename=package://six_dof/meshes/footfixedv3.stl scale=0.001 0.001 0.001
- link right_foot: geometry collision mesh filename=package://six_dof/meshes/footfixedv3.stl scale=0.001 0.001 0.001; visual mesh filename=package://six_dof/meshes/footfixedv3.stl scale=0.001 0.001 0.001
Joints:
- joint left_shin_foot: origin xyz=-0.027 -0.130 0 rpy=0 0 0 -> xyz=-0.02 -0.130 0 rpy=0 0 0
- joint left_thigh_shin: origin xyz=0.005 -0.160 0 rpy=0 0 0 -> xyz=-0.0425 -0.160 0 rpy=0 3.14 0

Commit message: resolved computeCollisions() import

File: src/six_dof/urdf/6dof_from_hip.urdf (robot description, URDF)
Before this commit: robot 6dof, 10 links, 9 joints
Joints:
- joint left_thigh_shin: limit lower=-0.52 upper=0.52 effort=35.0 velocity=0.1 -> lower=-1.04 upper=1.04 effort=35.0 velocity=0.1
- joint right_thigh_shin: limit lower=-0.52 upper=0.52 effort=35.0 velocity=0.1 -> lower=-1.04 upper=1.04 effort=35.0 velocity=0.1

Commit message: added inertial values for urdf

File: src/six_dof/urdf/6dof_from_hip.urdf (robot description, URDF)
Before this commit: robot 6dof, 10 links, 9 joints
Links:
- link body: mass None -> 0.9
- link left_foot: mass None -> 0.022566
- link left_shin: mass None -> 0.014172
- link left_thigh: mass None -> 0.067626
- link right_foot: mass None -> 0.022566
- link right_shin: mass None -> 0.014172
- link right_thigh: mass None -> 0.067538
