Commit message: addded imu sensor

File: src/six_dof/urdf/6dof_from_hip_control.urdf (robot description, URDF)
Before this commit: robot 6dof, 10 links, 9 joints
Links:
- added link imu_link, mass 0.000001
Joints:
- added joint body_to_imu: type fixed, parent body, child imu_link, origin xyz=0.065 -0.0 -0.047 rpy=0.0 -1.57 -1.57

Commit message: walks forward

File: src/six_dof/urdf/6dof_from_hip_control.urdf (robot description, URDF)
Before this commit: robot 6dof, 11 links, 10 joints
Links:
- link imu_link: mass 0.000001 -> 0.0001
