Commit message: added simplified meshes

File: src/six_dof/urdf/simplified_6dof_from_hip_control.urdf (robot description, URDF)
Before this commit: robot 6dof, 11 links, 10 joints
Links:
- link left_foot: geometry collision mesh filename=package://six_dof/meshes/convex_hull_stl/footfixedv3.stl scale=0.0001 0.0001 0.0001; visual mesh filename=package://six_dof/meshes/convex_hull_stl/footfixedv3.stl scale=0.0001 0.0001 0.0001
- link left_shin: geometry collision mesh filename=package://six_dof/meshes/convex_hull_stl/rightshinv3.stl scale=0.0001 0.0001 0.0001; visual mesh filename=package://six_dof/meshes/convex_hull_stl/rightshinv3.stl scale=0.0001 0.0001 0.0001
- link left_thigh: geometry collision mesh filename=package://six_dof/meshes/convex_hull_stl/leftthighfixedv1.s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 scale=0.0001 0.0001 0.0001; visual mesh filename=package://six_dof/meshes/convex_hull_stl/leftthighfixedv1.s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 scale=0.0001 0.0001 0.0001
- link right_foot: geometry collision mesh filename=package://six_dof/meshes/convex_hull_stl/footfixedv3.stl scale=0.0001 0.0001 0.0001; visual mesh filename=package://six_dof/meshes/convex_hull_stl/footfixedv3.stl scale=0.0001 0.0001 0.0001
- link right_shin: geometry collision mesh filename=package://six_dof/meshes/convex_hull_stl/rightshinfixedv2.s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 scale=0.0001 0.0001 0.0001; visual mesh filename=package://six_dof/meshes/convex_hull_stl/rightshinfixedv2.s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 scale=0.0001 0.0001 0.0001
- link right_thigh: geometry collision mesh filename=package://six_dof/meshes/convex_hull_stl/rightthighfixedv2.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 scale=0.0001 0.0001 0.0001; visual mesh filename=package://six_dof/meshes/convex_hull_stl/rightthighfixedv2.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 scale=0.0001 0.0001 0.0001
