Commit message: added convex hulls, position controller node

File: src/eight_dof/urdf/simplified_8dof_from_hip.urdf (robot description, URDF)
Before this commit: robot 8dof, 10 links, 9 joints
Links:
- link body: geometry collision mesh filename=package://eight_dof/meshes/convex_hull/body.stl scale=0.0001 0.0001 0.0001; visual mesh filename=package://eight_dof/meshes/convex_hull/body.stl scale=0.0001 0.0001 0.0001
- link left_foot: geometry collision mesh filename=package://eight_dof/meshes/convex_hull/foot.stl scale=0.0001 0.0001 0.0001; visual mesh filename=package://eight_dof/meshes/convex_hull/foot.stl scale=0.0001 0.0001 0.0001
- link left_shin: geometry collision mesh filename=package://eight_dof/meshes/convex_hull/shin.stl scale=0.00001 0.00001 0.00001; visual mesh filename=package://eight_dof/meshes/convex_hull/shin.stl scale=0.00001 0.00001 0.00001
- link left_thigh: geometry collision mesh filename=package://eight_dof/meshes/convex_hull/thigh.stl scale=0.00001 0.00001 0.00001; visual mesh filename=package://eight_dof/meshes/convex_hull/thigh.stl scale=0.00001 0.00001 0.00001
- link right_foot: geometry collision mesh filename=package://eight_dof/meshes/convex_hull/foot.stl scale=0.0001 0.0001 0.0001; visual mesh filename=package://eight_dof/meshes/convex_hull/foot.stl scale=0.0001 0.0001 0.0001
- link right_shin: geometry collision mesh filename=package://eight_dof/meshes/convex_hull/shin.stl scale=0.00001 0.00001 0.00001; visual mesh filename=package://eight_dof/meshes/convex_hull/shin.stl scale=0.00001 0.00001 0.00001
- link right_thigh: geometry collision mesh filename=package://eight_dof/meshes/convex_hull/thigh.stl scale=0.00001 0.00001 0.00001; visual mesh filename=package://eight_dof/meshes/convex_hull/thigh.stl scale=0.00001 0.00001 0.00001
