Commit message: working inertia model

File: src/eight_dof/urdf/8dof_from_hip.urdf (robot description, URDF)
Before this commit: robot 8dof, 10 links, 10 joints
Links:
- link body: mass None -> 2.343632
- link left_foot: mass None -> 0.414934; geometry collision mesh filename=package://eight_dof/meshes/foot.stl scale=0.0001 0.0001 0.0001; visual mesh filename=package://eight_dof/meshes/footv2.stl scale=0.0001 0.0001 0.0001
- link left_shin: mass None -> 1.507647
- link left_thigh: mass None -> 0.65958
- link right_foot: mass None -> 0.414934; geometry collision mesh filename=package://eight_dof/meshes/foot.stl scale=0.0001 0.0001 0.0001; visual mesh filename=package://eight_dof/meshes/footv2.stl scale=0.0001 0.0001 0.0001
- link right_shin: mass None -> 1.507647
- link right_thigh: mass None -> 0.65958
Joints:
- removed joint body_left_lateral
- removed joint body_right_lateral
- removed joint body_right_thigh
- removed joint left_intermediate_thigh
- removed joint right_intermediate_thigh
- added joint hip_left: type continuous, parent left_intermediate_link, child left_thigh, origin xyz=0.01 0.0 0.044 rpy=0.0 0.0 0.0, axis  1 0 0, limit effort=15.0 velocity=33.0
- added joint hip_left_lateral: type continuous, parent body, child left_intermediate_link, origin xyz=0.0897 0.0 0.0 rpy=0.0 0.0 0.0, axis  0 0 1, limit effort=15.0 velocity=33.0
- added joint hip_right: type continuous, parent right_intermediate_link, child right_thigh, origin xyz=-0.01 0.0 0.044 rpy=0.0 -3.14 0.0, axis  1 0 0, limit effort=15.0 velocity=33.0
- added joint hip_right_lateral: type continuous, parent body, child right_intermediate_link, origin xyz=-0.0897 0.0 0.0 rpy=0.0 0.0 0.0, axis  0 0 1, limit effort=15.0 velocity=33.0
- joint left_ankle: limit lower=-0.52 upper=0.52 effort=35.0 velocity=0.1 -> lower=-2.3 upper=2.3 effort=6.5 velocity=8.0
- joint left_knee: limit lower=-0.52 upper=0.52 effort=35.0 velocity=0.1 -> effort=15.0 velocity=33.0; type revolute -> continuous
- joint right_ankle: limit lower=-0.52 upper=0.52 effort=35.0 velocity=0.1 -> lower=-2.3 upper=2.3 effort=6.0 velocity=8.0
- joint right_knee: limit lower=-0.52 upper=0.52 effort=35.0 velocity=0.1 -> effort=15.0 velocity=33.0; type revolute -> continuous

Commit message: eight_dof walks in sim

File: src/eight_dof/urdf/8dof_from_hip.urdf (robot description, URDF)
Before this commit: robot 8dof, 10 links, 9 joints
Links:
- link body: mass 2.343632 -> 3.101495; geometry collision mesh filename=package://eight_dof/meshes/chassisv6.stl scale=0.0001 0.0001 0.0001; visual mesh filename=package://eight_dof/meshes/chassisv6.stl scale=0.0001 0.0001 0.0001
- link left_foot: mass 0.414934 -> 0.170956; geometry collision mesh filename=package://eight_dof/meshes/footv6.stl scale=0.001 0.001 0.001; visual mesh filename=package://eight_dof/meshes/footv6.stl scale=0.001 0.001 0.001
- link left_shin: mass 1.507647 -> 1.488501; geometry collision mesh filename=package://eight_dof/meshes/shinv4.stl scale=0.001 0.001 0.001; visual mesh filename=package://eight_dof/meshes/shinv4.stl scale=0.001 0.001 0.001
- link left_thigh: geometry collision mesh filename=package://eight_dof/meshes/thighv3.stl scale=0.000001 0.000001 0.000001; visual mesh filename=package://eight_dof/meshes/thighv3.stl scale=0.000001 0.000001 0.000001
- link right_foot: mass 0.414934 -> 0.170956; geometry collision mesh filename=package://eight_dof/meshes/footv6.stl scale=0.001 0.001 0.001; visual mesh filename=package://eight_dof/meshes/footv6.stl scale=0.001 0.001 0.001
- link right_shin: mass 1.507647 -> 1.488501; geometry collision mesh filename=package://eight_dof/meshes/shinv4.stl scale=0.001 0.001 0.001; visual mesh filename=package://eight_dof/meshes/shinv4.stl scale=0.001 0.001 0.001
- link right_thigh: geometry collision mesh filename=package://eight_dof/meshes/thighv3.stl scale=0.000001 0.000001 0.000001; visual mesh filename=package://eight_dof/meshes/thighv3.stl scale=0.000001 0.000001 0.000001
Joints:
- joint left_ankle: origin xyz=0.02 -0.244 0.0 rpy=0.0 0.0 0.0 -> xyz=0.02 -0.315 0.0 rpy=0.0 0.0 0.0
- joint right_ankle: origin xyz=0.02 -0.244 0.0 rpy=0.0 -3.14 0.0 -> xyz=0.02 -0.315 0.0 rpy=0.0 -3.14 0.0

File: src/eight_dof/urdf/simplified_8dof_from_hip.urdf (robot description, URDF)
Before this commit: robot 8dof, 10 links, 9 joints
Links:
- link body: mass 2.343632 -> 3.101495; geometry collision mesh filename=package://eight_dof/meshes/chassisv6.stl scale=0.0001 0.0001 0.0001; visual mesh filename=package://eight_dof/meshes/chassisv6.stl scale=0.0001 0.0001 0.0001
- link left_foot: mass 0.414934 -> 0.170956; geometry collision mesh filename=package://eight_dof/meshes/footv6.stl scale=0.001 0.001 0.001; visual mesh filename=package://eight_dof/meshes/footv6.stl scale=0.001 0.001 0.001
- link left_shin: mass 1.507647 -> 1.488501; geometry collision mesh filename=package://eight_dof/meshes/shinv4.stl scale=0.001 0.001 0.001; visual mesh filename=package://eight_dof/meshes/shinv4.stl scale=0.001 0.001 0.001
- link left_thigh: geometry collision mesh filename=package://eight_dof/meshes/thighv3.stl scale=0.000001 0.000001 0.000001; visual mesh filename=package://eight_dof/meshes/thighv3.stl scale=0.000001 0.000001 0.000001
- link right_foot: mass 0.414934 -> 0.170956; geometry collision mesh filename=package://eight_dof/meshes/footv6.stl scale=0.001 0.001 0.001; visual mesh filename=package://eight_dof/meshes/footv6.stl scale=0.001 0.001 0.001
- link right_shin: mass 1.507647 -> 1.488501; geometry collision mesh filename=package://eight_dof/meshes/shinv4.stl scale=0.001 0.001 0.001; visual mesh filename=package://eight_dof/meshes/shinv4.stl scale=0.001 0.001 0.001
- link right_thigh: geometry collision mesh filename=package://eight_dof/meshes/thighv3.stl scale=0.000001 0.000001 0.000001; visual mesh filename=package://eight_dof/meshes/thighv3.stl scale=0.000001 0.000001 0.000001
Joints:
- joint left_ankle: origin xyz=0.02 -0.244 0.0 rpy=0.0 0.0 0.0 -> xyz=0.02 -0.315 0.0 rpy=0.0 0.0 0.0
- joint right_ankle: origin xyz=0.02 -0.244 0.0 rpy=0.0 -3.14 0.0 -> xyz=0.02 -0.315 0.0 rpy=0.0 -3.14 0.0

Commit message: added new convex hulls for eight dof

File: src/eight_dof/urdf/8dof_from_hip.urdf (robot description, URDF)
Before this commit: robot 8dof, 10 links, 9 joints
Joints:
- joint left_ankle: origin xyz=0.02 -0.315 0.0 rpy=0.0 0.0 0.0 -> xyz=0.02 -0.317 0.0 rpy=0.0 0.0 0.0
- joint right_ankle: origin xyz=0.02 -0.315 0.0 rpy=0.0 -3.14 0.0 -> xyz=0.02 -0.317 0.0 rpy=0.0 -3.14 0.0

File: src/eight_dof/urdf/simplified_8dof_from_hip.urdf (robot description, URDF)
Before this commit: robot 8dof, 10 links, 9 joints
Links:
- link body: geometry collision mesh filename=package://eight_dof/meshes/convex_hull/bodyv2.stl scale=0.0001 0.0001 0.0001; visual mesh filename=package://eight_dof/meshes/convex_hull/bodyv2.stl scale=0.0001 0.0001 0.0001
- link left_foot: geometry collision mesh filename=package://eight_dof/meshes/convex_hull/footv2.stl scale=0.001 0.001 0.001; visual mesh filename=package://eight_dof/meshes/convex_hull/footv2.stl scale=0.001 0.001 0.001
- link left_shin: geometry collision mesh filename=package://eight_dof/meshes/convex_hull/shinv2.stl scale=0.001 0.001 0.001; visual mesh filename=package://eight_dof/meshes/convex_hull/shinv2.stl scale=0.001 0.001 0.001
- link left_thigh: geometry collision mesh filename=package://eight_dof/meshes/convex_hull/thighv2.stl scale=0.000001 0.000001 0.000001; visual mesh filename=package://eight_dof/meshes/convex_hull/thighv2.stl scale=0.000001 0.000001 0.000001
- link right_foot: geometry collision mesh filename=package://eight_dof/meshes/convex_hull/footv2.stl scale=0.001 0.001 0.001; visual mesh filename=package://eight_dof/meshes/convex_hull/footv2.stl scale=0.001 0.001 0.001
- link right_shin: geometry collision mesh filename=package://eight_dof/meshes/convex_hull/shinv2.stl scale=0.001 0.001 0.001; visual mesh filename=package://eight_dof/meshes/convex_hull/shinv2.stl scale=0.001 0.001 0.001
- link right_thigh: geometry collision mesh filename=package://eight_dof/meshes/convex_hull/thighv2.stl scale=0.000001 0.000001 0.000001; visual mesh filename=package://eight_dof/meshes/convex_hull/thighv2.stl scale=0.000001 0.000001 0.000001
Joints:
- joint left_ankle: origin xyz=0.02 -0.315 0.0 rpy=0.0 0.0 0.0 -> xyz=0.02 -0.330 0.0 rpy=0.0 0.0 0.0
- joint right_ankle: origin xyz=0.02 -0.315 0.0 rpy=0.0 -3.14 0.0 -> xyz=0.02 -0.330 0.0 rpy=0.0 -3.14 0.0

Commit message: added chassis with no battery

File: src/eight_dof/urdf/8dof_from_hip.urdf (robot description, URDF)
Before this commit: robot 8dof, 10 links, 9 joints
Links:
- link body: mass 3.101495 -> 1.900281; geometry collision mesh filename=package://eight_dof/meshes/chassisv6.stl scale=0.001 0.001 0.001; visual mesh filename=package://eight_dof/meshes/chassis_no_batt.stl scale=0.001 0.001 0.001

File: src/eight_dof/urdf/simplified_8dof_from_hip.urdf (robot description, URDF)
Before this commit: robot 8dof, 10 links, 9 joints
Links:
- link body: mass 3.101495 -> 1.900281; geometry collision mesh filename=package://eight_dof/meshes/convex_hull/chassis_no_batt.stl scale=0.001 0.001 0.001; visual mesh filename=package://eight_dof/meshes/convex_hull/chassis_no_batt.stl scale=0.001 0.001 0.001
